Commit message: Update ROS2 workspace: update navigation configs, URDF models, and add new automation scripts

File: src/my_factory/urdf/gazebo_control.xacro (robot description, xacro)
@@ -8,21 +8,26 @@
             <right_joint>front_right_wheel_joint</right_joint>
             <right_joint>back_right_wheel_joint</right_joint>
-            <wheel_separation>2.1</wheel_separation>
-            <wheel_diameter>0.3</wheel_diameter>
+            <wheel_separation>0.84</wheel_separation>
+            <wheel_diameter>0.20</wheel_diameter>
             <max_wheel_torque>60</max_wheel_torque>
             <max_wheel_acceleration>2.0</max_wheel_acceleration>
             <max_linear_acceleration>1.0</max_linear_acceleration>
             <max_angular_acceleration>1.5</max_angular_acceleration>
-            <topic>cmd_vel</topic>
+            <topic>/cmd_vel</topic>
             <frame_id>odom</frame_id>
             <child_frame_id>base_footprint</child_frame_id>
-            <publish_odom>true</publish_odom>
+            <odom_topic>trash_odom</odom_topic>
             <publish_odom_tf>false</publish_odom_tf>
             <publish_wheel_tf>false</publish_wheel_tf>
-            <use_sim_time>true</use_sim_time>
-            <update_rate>50</update_rate>
+        </plugin>
+        <plugin filename="ignition-gazebo-odometry-publisher-system" name="ignition::gazebo::systems::OdometryPublisher">
+            <odom_frame>odom</odom_frame>
+            <robot_base_frame>base_footprint</robot_base_frame>
+            <odom_publish_frequency>50</odom_publish_frequency>
+            <odom_topic>/model/warehouse_robot/odometry</odom_topic>
+            <dimensions>2</dimensions>
         </plugin>
         <plugin filename="ignition-gazebo-joint-state-publisher-system" name="ignition::gazebo::systems::JointStatePublisher">
-            <topic>joint_states</topic>
+            <topic>/joint_states</topic>
             <joint_name>front_left_wheel_joint</joint_name>
             <joint_name>front_right_wheel_joint</joint_name>

File: src/my_factory/urdf/lidar.xacro (robot description, xacro)
@@ -5,5 +5,5 @@
             <parent link="base_link"/>
             <child link="${prefix}_bracket"/>
-            <origin xyz="${x_pos * 0.98} ${y_pos * 0.98} ${z_pos - 0.02}" rpy="0 0 ${rotation}"/>
+            <origin xyz="${x_pos} ${y_pos} ${z_pos}" rpy="0 0 ${rotation}"/>
         </joint>
         <link name="${prefix}_bracket">
@@ -44,11 +44,11 @@
                             <samples>360</samples>
                             <resolution>1</resolution>
-                            <min_angle>-3.14</min_angle>
-                            <max_angle>3.14</max_angle>
+                            <min_angle>-3.14159</min_angle>
+                            <max_angle>3.14159</max_angle>
                         </horizontal>
                     </scan>
                     <range>
                         <min>0.3</min>
-                        <max>12.0</max>
+                        <max>60.0</max>
                         <resolution>0.01</resolution>
                     </range>
@@ -59,5 +59,4 @@
         </gazebo>
     </xacro:macro>
-    <xacro:lidar prefix="front_right" x_pos="1.0" y_pos="-1.0" z_pos="0.27" rotation="${-pi/4}"/>
-    <xacro:lidar prefix="back_left" x_pos="-1.0" y_pos="1.0" z_pos="0.27" rotation="${3*pi/4}"/>
-</robot>
+    <xacro:lidar prefix="front_right" x_pos="-0.36" y_pos="0.0" z_pos="0.92" rotation="0.0"/>
+    </robot>

File: src/my_factory/urdf/mobile_base.xacro (robot description, xacro)
@@ -1,18 +1,18 @@
 <?xml version="1.0"?>
 <robot xmlns:xacro="http://www.ros.org/wiki/xacro">
-    <xacro:property name="base_length" value="2.0"/>
-    <xacro:property name="base_width" value="2.0"/>
+    <xacro:property name="base_length" value="0.8"/>
+    <xacro:property name="base_width" value="0.8"/>
     <xacro:property name="base_height" value="0.1"/>
-    <xacro:property name="wheel_radius" value="0.15"/>
+    <xacro:property name="wheel_radius" value="0.10"/>
     <xacro:property name="base_z_offset" value="${wheel_radius}"/>
-    <xacro:property name="wheel_thickness" value="0.08"/>
-    <xacro:property name="wheel_offset_x" value="0.8"/>
-    <xacro:property name="wheel_offset_y" value="1.05"/>
-    <xacro:property name="pillar_height" value="2.0"/>
-    <xacro:property name="pillar_side" value="0.08"/>
-    <xacro:property name="pillar_offset_x" value="0.9"/>
-    <xacro:property name="pillar_offset_y" value="0.9"/>
-    <xacro:property name="bar_radius" value="0.015"/>
-    <xacro:property name="bar_length" value="1.8"/>
+    <xacro:property name="wheel_thickness" value="0.05"/>
+    <xacro:property name="wheel_offset_x" value="0.32"/>
+    <xacro:property name="wheel_offset_y" value="0.42"/>
+    <xacro:property name="pillar_height" value="0.8"/>
+    <xacro:property name="pillar_side" value="0.04"/>
+    <xacro:property name="pillar_offset_x" value="0.36"/>
+    <xacro:property name="pillar_offset_y" value="0.36"/>
+    <xacro:property name="bar_radius" value="0.01"/>
+    <xacro:property name="bar_length" value="0.72"/>
     <link name="base_footprint"/>
     <joint name="base_joint" type="fixed">
@@ -31,5 +31,5 @@
             <origin xyz="0 0 ${base_height/2}" rpy="0 0 0"/>
         </collision>
-        <xacro:inertial_box mass="50.0" x="${base_length}" y="${base_width}" z="${base_height}">
+        <xacro:inertial_box mass="15.0" x="${base_length}" y="${base_width}" z="${base_height}">
             <origin xyz="0 0 ${base_height/2}" rpy="0 0 0"/>
         </xacro:inertial_box>
@@ -46,5 +46,5 @@
                 <origin xyz="0 0 0" rpy="${pi/2} 0 0"/>
             </collision>
-            <xacro:inertial_cylinder mass="2.0" length="${wheel_thickness}" radius="${wheel_radius}">
+            <xacro:inertial_cylinder mass="0.5" length="${wheel_thickness}" radius="${wheel_radius}">
                 <origin xyz="0 0 0" rpy="${pi/2} 0 0"/>
             </xacro:inertial_cylinder>
@@ -62,5 +62,5 @@
             <visual> <geometry> <box size="${pillar_side} ${pillar_side} ${pillar_height}"/> </geometry> <material name="white"/> </visual>
             <collision> <geometry> <box size="${pillar_side} ${pillar_side} ${pillar_height}"/> </geometry> </collision>
-            <xacro:inertial_box mass="1.0" x="${pillar_side}" y="${pillar_side}" z="${pillar_height}">
+            <xacro:inertial_box mass="0.2" x="${pillar_side}" y="${pillar_side}" z="${pillar_height}">
                 <origin xyz="0 0 0" rpy="0 0 0"/>
             </xacro:inertial_box>
@@ -76,5 +76,5 @@
             <visual> <geometry> <cylinder radius="${bar_radius}" length="${length}"/> </geometry> <material name="white"/> </visual>
             <collision> <geometry> <cylinder radius="${bar_radius}" length="${length}"/> </geometry> </collision>
-            <xacro:inertial_cylinder mass="0.5" length="${length}" radius="${bar_radius}">
+            <xacro:inertial_cylinder mass="0.1" length="${length}" radius="${bar_radius}">
                 <origin xyz="0 0 0" rpy="0 0 0"/>
             </xacro:inertial_cylinder>
@@ -99,6 +99,7 @@
     <xacro:macro name="wheel_gazebo" params="prefix">
         <gazebo reference="${prefix}_wheel">
-            <mu1 value="100.0"/>
-            <mu2 value="100.0"/>
+            <mu1 value="0.2"/>
+            <mu2 value="0.2"/>
+            <fdir1 value="1 0 0"/>
             <kp value="1000000.0"/>
             <kd value="10.0"/>

File: src/my_factory/urdf/my_robot.urdf.xacro (robot description, xacro)
@@ -1,15 +1,10 @@
 <?xml version="1.0"?>
 <robot xmlns:xacro="http://www.ros.org/wiki/xacro" name="my_robot">
-    <!-- 1. استدعاء الخصائص المشتركة والألوان -->
     <xacro:include filename="common_properties.xacro"/>
-    <!-- 2. استدعاء هيكل الروبوت (تأكد أن base_link هو الأب الرئيسي هنا) -->
     <xacro:include filename="mobile_base.xacro"/>
-    <!-- 3. استدعاء الحساسات (Lidar) -->
     <xacro:include filename="lidar.xacro"/>
-    <!-- 4. استدعاء متحكمات الغازيبو -->
+    <xacro:include filename="camera.xacro"/>
     <xacro:include filename="gazebo_control.xacro"/>
-    <!-- إعدادات Ignition Gazebo لضمان استقرار شجرة الـ TF -->
     <gazebo>
-        <!-- هذا البلجن يضمن أن غازيبو يرسل وضعية الروبوت الحقيقية إلى ROS -->
         <plugin filename="ignition-gazebo-pose-publisher-system" name="ignition::gazebo::systems::PosePublisher">
             <publish_link_pose>true</publish_link_pose>
@@ -20,5 +15,5 @@
             <static_publisher>true</static_publisher>
             <static_update_frequency>100</static_update_frequency>
-        </plugin>
+       </plugin>
     </gazebo>
 </robot>

File: src/my_factory/urdf/panda_ign.urdf.xacro (robot description, xacro)
@@ -1,11 +1,4 @@
 <?xml version="1.0"?>
 <robot xmlns:xacro="http://www.ros.org/wiki/xacro" name="panda">
-    <!--
-      Ignition-ready Panda for ign_ros2_control + MoveIt.
-      The MoveIt panda description (moveit_resources_panda_description) is purely
-      visual/kinematic (no <inertial>), so this file re-declares the chain with the
-      same meshes/origins/limits PLUS approximate Franka link inertials and a fixed
-      'world' base so the arm can be simulated under physics.
-    -->
     <xacro:property name="mesh_pkg" value="package://moveit_resources_panda_description/meshes"/>
     <xacro:macro name="panda_inertial" params="mass inertia">
@@ -16,10 +9,9 @@
         </inertial>
     </xacro:macro>
-    <!-- Fixed base: anchor the arm to the world at the origin on the floor -->
     <link name="world"/>
     <joint name="panda_world_joint" type="fixed">
         <parent link="world"/>
         <child link="panda_link0"/>
-        <origin xyz="0 0 0" rpy="0 0 0"/>
+        <origin xyz="5.36 -16.9 0.11" rpy="0 0 0"/>
     </joint>
     <link name="panda_link0">
@@ -38,5 +30,5 @@
         <axis xyz="0 0 1"/>
         <limit effort="87" lower="-2.9671" upper="2.9671" velocity="2.3925"/>
-        <dynamics damping="1.0" friction="0.0"/>
+        <dynamics damping="10.0" friction="1.0"/>
     </joint>
     <link name="panda_link2">
@@ -50,5 +42,5 @@
         <axis xyz="0 0 1"/>
         <limit effort="87" lower="-1.8326" upper="1.8326" velocity="2.3925"/>
-        <dynamics damping="1.0" friction="0.0"/>
+        <dynamics damping="10.0" friction="1.0"/>
     </joint>
     <link name="panda_link3">
@@ -62,5 +54,5 @@
         <axis xyz="0 0 1"/>
         <limit effort="87" lower="-2.9671" upper="2.9671" velocity="2.3925"/>
-        <dynamics damping="1.0" friction="0.0"/>
+        <dynamics damping="10.0" friction="1.0"/>
     </joint>
     <link name="panda_link4">
@@ -74,5 +66,5 @@
         <axis xyz="0 0 1"/>
         <limit effort="87" lower="-3.1416" upper="0.0873" velocity="2.3925"/>
-        <dynamics damping="1.0" friction="0.0"/>
+        <dynamics damping="10.0" friction="1.0"/>
     </joint>
     <link name="panda_link5">
@@ -86,5 +78,5 @@
         <axis xyz="0 0 1"/>
         <limit effort="12" lower="-2.9671" upper="2.9671" velocity="2.8710"/>
-        <dynamics damping="1.0" friction="0.0"/>
+        <dynamics damping="10.0" friction="1.0"/>
     </joint>
     <link name="panda_link6">
@@ -98,5 +90,5 @@
         <axis xyz="0 0 1"/>
         <limit effort="12" lower="-0.0873" upper="3.8223" velocity="2.8710"/>
-        <dynamics damping="1.0" friction="0.0"/>
+        <dynamics damping="10.0" friction="1.0"/>
     </joint>
     <link name="panda_link7">
@@ -110,5 +102,5 @@
         <axis xyz="0 0 1"/>
         <limit effort="12" lower="-2.9671" upper="2.9671" velocity="2.8710"/>
-        <dynamics damping="1.0" friction="0.0"/>
+        <dynamics damping="10.0" friction="1.0"/>
     </joint>
     <link name="panda_link8">
@@ -149,5 +141,5 @@
         <axis xyz="0 1 0"/>
         <limit effort="20" lower="0.0" upper="0.04" velocity="0.2"/>
-        <dynamics damping="1.0" friction="0.0"/>
+        <dynamics damping="10.0" friction="0.0"/>
     </joint>
     <joint name="panda_finger_joint2" type="prismatic">
@@ -157,10 +149,9 @@
         <limit effort="20" lower="0.0" upper="0.04" velocity="0.2"/>
         <mimic joint="panda_finger_joint1"/>
-        <dynamics damping="1.0" friction="0.0"/>
-    </joint>
-    <!-- ros2_control: Ignition hardware -->
-    <ros2_control name="PandaIgnitionSystem" type="system">
+        <dynamics damping="10.0" friction="0.0"/>
+    </joint>
+    <ros2_control name="PandaGazeboSystem" type="system">
         <hardware>
-            <plugin>ign_ros2_control/IgnitionSystem</plugin>
+            <plugin>gz_ros2_control/GazeboSimSystem</plugin>
         </hardware>
         <xacro:macro name="arm_joint_ctrl" params="jname init">
@@ -185,6 +176,4 @@
             <state_interface name="effort"/>
         </joint>
-        <!-- ign_ros2_control mirrors this joint from finger_joint1 via the 'mimic' param
-             (it does NOT read the URDF <mimic> tag), so it must be declared here. -->
         <joint name="panda_finger_joint2">
             <param name="mimic">panda_finger_joint1</param>
@@ -196,9 +185,61 @@
         </joint>
     </ros2_control>
-    <!-- ign_ros2_control system plugin: runs the controller_manager inside Ignition -->
     <gazebo>
-        <plugin filename="ign_ros2_control-system" name="ign_ros2_control::IgnitionROS2ControlPlugin">
+        <plugin filename="libgz_ros2_control-system.so" name="gz_ros2_control::GazeboSimROS2ControlPlugin">
             <parameters>$(find my_factory)/config/panda_controllers.yaml</parameters>
-            <controller_manager_node_name>controller_manager</controller_manager_node_name>
+            <robot_param_node>/panda/robot_state_publisher</robot_param_node>
+            <controller_manager_node_name>/controller_manager</controller_manager_node_name>
+            <ros>
+                <remapping>/joint_states:=/panda/joint_states</remapping>
+            </ros>
+        </plugin>
+    </gazebo>
+    <!-- ========================================== -->
+    <!-- 🟢 إضافة كاميرا السقف الثابتة فوق المكعب مباشرة -->
+    <!-- ========================================== -->
+    <link name="camera_link">
+        <visual>
+            <geometry>
+                <box size="0.04 0.04 0.04"/> <!-- كبرتها قليلاً لتراها بوضوح في المحاكي -->
+            </geometry>
+            <material name="black">
+                <color rgba="0.1 0.1 0.1 1.0"/>
+            </material>
+        </visual>
+        <collision>
+            <geometry>
+                <box size="0.04 0.04 0.04"/>
+            </geometry>
+        </collision>
+        <xacro:panda_inertial mass="0.05" inertia="0.0001"/>
+    </link>
+    <!-- 🛠️ تم التعديل: ربط الكاميرا بالعالم (world) مباشرة لسهولة وضع الإحداثيات -->
+    <joint name="camera_joint" type="fixed">
+        <parent link="world"/>
+        <child link="camera_link"/>
+        <!-- إحداثيات المكعب + 70 سم ارتفاع (Z = 0.36 + 0.70 = 1.06) والنظر لأسفل بزاوية 90 درجة (Pitch = 1.5708) -->
+        <origin xyz="6.0 -16.8 1.06" rpy="0 1.5708 0"/>
+    </joint>
+    <gazebo reference="camera_link">
+        <sensor name="panda_camera" type="rgbd">
+            <camera>
+                <horizontal_fov>1.047</horizontal_fov>
+                <image>
+                    <width>640</width>
+                    <height>480</height>
+                    <format>R8G8B8</format>
+                </image>
+                <clip>
+                    <near>0.01</near>
+                    <far>20.0</far>
+                </clip>
+            </camera>
+            <always_on>1</always_on>
+            <update_rate>30.0</update_rate>
+            <visualize>true</visualize>
+            <topic>camera/image_raw</topic>
+        </sensor>
+        <plugin filename="libignition-gazebo-sensors-system.so" name="ignition::gazebo::systems::Sensors">
+            <render_engine>ogre2</render_engine>
         </plugin>
     </gazebo>
