Commit message: اكتب هنا وصفاً مختصراً للتعديلات التي فعلتها

File: src/my_factory/urdf/camera.xacro (robot description, xacro)
@@ -1,10 +1,12 @@
 <?xml version="1.0"?>
 <robot xmlns:xacro="http://www.ros.org/wiki/xacro">
-    <joint name="camera_joint" type="fixed">
+    <!-- 🟢 تم تغيير الاسم إلى base_camera_joint -->
+    <joint name="base_camera_joint" type="fixed">
         <parent link="base_link"/>
-        <child link="camera_link"/>
+        <child link="base_camera_link"/>
         <origin xyz="0.38 0.0 0.115" rpy="0 0 0"/>
     </joint>
-    <link name="camera_link">
+    <!-- 🟢 تم تغيير الاسم إلى base_camera_link -->
+    <link name="base_camera_link">
         <visual>
             <geometry> <box size="0.03 0.1 0.03"/> </geometry>
@@ -18,19 +20,20 @@
         </xacro:inertial_box>
     </link>
-    <joint name="camera_depth_joint" type="fixed">
-        <parent link="camera_link"/>
-        <child link="camera_depth_frame"/>
-        <!-- 🟢 الزوايا أصفار لكي ينظر للأمام مباشرة -->
+    <!-- 🟢 تم تغيير الاسم إلى base_camera_depth_joint وربطه بالروابط الجديدة -->
+    <joint name="base_camera_depth_joint" type="fixed">
+        <parent link="base_camera_link"/>
+        <child link="base_camera_depth_frame"/>
         <origin xyz="0 0 0" rpy="0 0 0"/>
     </joint>
-    <link name="camera_depth_frame"/>
-    <gazebo reference="camera_link">
+    <link name="base_camera_depth_frame"/>
+    <!-- 🟢 تحديث المرجع ليتوافق مع الرابط الجديد -->
+    <gazebo reference="base_camera_link">
         <sensor name="depth_camera" type="gpu_lidar">
             <always_on>1</always_on>
             <update_rate>5.0</update_rate>
             <visualize>true</visualize>
-            <topic>camera</topic>
-            <!-- 🟢 تم إرجاع الإطار الوهمي لتفادي انهيار جازيبو واختفاء الخريطة -->
-            <gz_frame_id>camera_depth_frame</gz_frame_id>
+            <topic>/base_camera/scan</topic>
+            <!-- 🟢 تحديث الإطار الوهمي لليدار -->
+            <gz_frame_id>base_camera_depth_frame</gz_frame_id>
             <lidar>
                 <scan>
@@ -44,7 +47,7 @@
                         <samples>10</samples>
                         <resolution>1</resolution>
-                        <!-- 🟢 الزاوية السالبة هنا تجعله ينظر للأسفل نحو الصناديق -->
-                        <min_angle>-0.4</min_angle>
-                        <max_angle>0.1</max_angle>
+                        <!-- 🟢 تم تعديل الزوايا لتتجنب الأرض وترصد الصناديق المنخفضة -->
+                        <min_angle>-0.05</min_angle>
+                        <max_angle>0.2</max_angle>
                     </vertical>
                 </scan>

File: src/my_factory/urdf/panda_ign.urdf.xacro (robot description, xacro)
@@ -195,52 +195,5 @@
         </plugin>
     </gazebo>
-    <!-- ========================================== -->
-    <!-- 🟢 إضافة كاميرا السقف الثابتة فوق المكعب مباشرة -->
-    <!-- ========================================== -->
-    <link name="camera_link">
-        <visual>
-            <geometry>
-                <box size="0.04 0.04 0.04"/> <!-- كبرتها قليلاً لتراها بوضوح في المحاكي -->
-            </geometry>
-            <material name="black">
-                <color rgba="0.1 0.1 0.1 1.0"/>
-            </material>
-        </visual>
-        <collision>
-            <geometry>
-                <box size="0.04 0.04 0.04"/>
-            </geometry>
-        </collision>
-        <xacro:panda_inertial mass="0.05" inertia="0.0001"/>
-    </link>
-    <!-- 🛠️ تم التعديل: ربط الكاميرا بالعالم (world) مباشرة لسهولة وضع الإحداثيات -->
-    <joint name="camera_joint" type="fixed">
-        <parent link="world"/>
-        <child link="camera_link"/>
-        <!-- إحداثيات المكعب + 70 سم ارتفاع (Z = 0.36 + 0.70 = 1.06) والنظر لأسفل بزاوية 90 درجة (Pitch = 1.5708) -->
-        <origin xyz="6.0 -16.8 1.06" rpy="0 1.5708 0"/>
-    </joint>
-    <gazebo reference="camera_link">
-        <sensor name="panda_camera" type="rgbd">
-            <camera>
-                <horizontal_fov>1.047</horizontal_fov>
-                <image>
-                    <width>640</width>
-                    <height>480</height>
-                    <format>R8G8B8</format>
-                </image>
-                <clip>
-                    <near>0.01</near>
-                    <far>20.0</far>
-                </clip>
-            </camera>
-            <always_on>1</always_on>
-            <update_rate>30.0</update_rate>
-            <visualize>true</visualize>
-            <topic>camera/image_raw</topic>
-        </sensor>
-        <plugin filename="libignition-gazebo-sensors-system.so" name="ignition::gazebo::systems::Sensors">
-            <render_engine>ogre2</render_engine>
-        </plugin>
-    </gazebo>
+    <!-- 🟢 استدعاء ملف كاميرا الذراع السقفية -->
+    <xacro:include filename="arm_camera.xacro"/>
 </robot>
